Commit message: add world and all launch file gazebo

File: description/base_robot.xacro (robot description, xacro)
@@ -1,5 +1,5 @@
 <?xml version="1.0"?>
 <robot xmlns:xacro="http://www.ros.org/wiki/xacro">
-    xacro:<xacro:include filename="inertial_macros.xacro" />
+  <xacro:include filename="inertial_macros.xacro"/>
   <!-- Define material only once -->
     <material name="white">
@@ -28,8 +28,12 @@
             </geometry>
             <origin xyz="0 0 0.1" rpy="0 0 0"/>
-            <!-- Apply material -->
-            <material name="white"/>
         </collision>
+        <xacro:inertial_box mass="0.5" x="0.6" y="0.4" z="0.2">
+          <origin xyz="0 0 0.1" rpy="0 0 0"/>
+        </xacro:inertial_box>
     </link>
+    <gazebo reference="base_link">
+        <material>Gazebo/White</material>
+    </gazebo>
     <link name="lidar">
         <visual>
@@ -37,5 +41,5 @@
                 <cylinder radius="0.1" length="0.05"/>
             </geometry>
-            <origin xyz="0 0 0" rpy="0 0 0" />
+            <origin xyz="0 0 0" rpy="0 0 0"/>
             <material name="black"/>
         </visual>
@@ -44,14 +48,40 @@
                 <cylinder radius="0.1" length="0.05"/>
             </geometry>
-            <origin xyz="0 0 0" rpy="0 0 0" />
-            <material name="black"/>
+            <origin xyz="0 0 0" rpy="0 0 0"/>
         </collision>
+        <xacro:inertial_cylinder mass="0.2" radius="0.1" length="0.05">
+              <origin xyz="0 0 0" rpy="0 0 0"/>
+        </xacro:inertial_cylinder>
     </link>
+    <gazebo reference="lidar">
+        <material>Gazebo/Black</material>
+    </gazebo>
     <link name="whil_wright">
+      <visual>
+          <geometry>
+            <cylinder radius="0.1" length="0.05"/>
+          </geometry>
+        <origin xyz="0 0 0" rpy="1.57 0 0"/>
+        <material name="blue"/>
+      </visual>
+      <collision>
+        <geometry>
+          <cylinder radius="0.1" length="0.05"/>
+        </geometry>
+        <origin xyz="0 0 0" rpy="1.57 0 0"/>
+      </collision>
+      <xacro:inertial_cylinder mass="0.2" radius="0.1" length="0.05">
+        <origin xyz="0 0 0" rpy="1.57 0 0"/>
+      </xacro:inertial_cylinder>
+    </link>
+    <gazebo reference="whil_wright">
+        <material>Gazebo/Blue</material>
+    </gazebo>
+    <link name="whil_left">
         <visual>
             <geometry>
                 <cylinder radius="0.1" length="0.05"/>
             </geometry>
-            <origin xyz="0 0 0" rpy="1.57 0 0 "/>
+            <origin xyz="0 0 0" rpy="1.57 0 0"/>
             <material name="blue"/>
         </visual>
@@ -60,24 +90,13 @@
                 <cylinder radius="0.1" length="0.05"/>
             </geometry>
-            <origin xyz="0 0 0" rpy="1.57 0 0 "/>
-            <material name="blue"/>
+            <origin xyz="0 0 0" rpy="1.57 0 0"/>
         </collision>
+        <xacro:inertial_cylinder mass="0.2" radius="0.1" length="0.05">
+          <origin xyz="0 0 0" rpy="1.57 0 0"/>
+        </xacro:inertial_cylinder>
     </link>
-    <link name="whil_left">
-        <visual>
-            <geometry>
-                <cylinder radius="0.1" length="0.05"/>
-            </geometry>
-            <origin xyz="0 0 0" rpy="1.57 0 0 "/>
-            <material name="blue"/>
-        </visual>
-        <collision>
-            <geometry>
-                <cylinder radius="0.1" length="0.05"/>
-            </geometry>
-            <origin xyz="0 0 0" rpy="1.57 0 0 "/>
-            <material name="blue"/>
-        </collision>
-    </link>
+    <gazebo reference="whil_left">
+        <material>Gazebo/Blue</material>
+    </gazebo>
     <link name="first_while">
         <visual>
@@ -93,5 +112,13 @@
             <origin xyz="0 0 0"/>
         </collision>
+        <xacro:inertial_sphere mass="0.1" radius="0.05">
+          <origin xyz="0.0 0.0 0.0"/>
+        </xacro:inertial_sphere>
     </link>
+    <gazebo reference="first_while">
+        <material>Gazebo/Red</material>
+        <mu1 value="0.001"/>
+        <mu2 value="0.001"/>
+    </gazebo>
 <!--lllllllllllllllllllllllllllllllllllllllllllllllllllllllllllllllllllllllink eded lllllllllllllllllllllllllllllllllll-->
     <joint name="base_lidar_joint" type="fixed">
@@ -103,5 +130,5 @@
         <parent link="base_link"/>
         <child link="whil_wright"/>
-        <origin xyz="-0.15 -0.225 0 " rpy="0 0 0"/>
+        <origin xyz="-0.15 -0.225 0" rpy="0 0 0"/>
         <axis xyz="0 1 0"/>
     </joint>
@@ -109,5 +136,5 @@
         <parent link="base_link"/>
         <child link="whil_left"/>
-        <origin xyz="-0.15 0.225 0 " rpy="0 0 0"/>
+        <origin xyz="-0.15 0.225 0" rpy="0 0 0"/>
         <axis xyz="0 1 0"/>
     </joint>

File: description/robot.urdf.xacro (robot description, xacro)
@@ -1,7 +1,5 @@
 <?xml version="1.0"?>
 <robot xmlns:xacro="http://www.ros.org/wiki/xacro" name="robot">
-  <!-- Include other xacro files -->
-  <xacro:include filename="$(find my_bot)/description/base.urdf.xacro" />
-  <!-- Later you can add more includes like wheels, sensors, arms, etc. -->
-  <!-- <xacro:include filename="$(find my_bot)/description/wheel.urdf.xacro" /> -->
+  <xacro:include filename="base_robot.xacro" />
+  <xacro:include filename="gazebo_control.xacro" />
 </robot>

Commit message: creat ros_controller and joystick launch fil

File: description/base_robot.xacro (robot description, xacro)
@@ -11,4 +11,10 @@
     <material name="blue">
         <color rgba="0 0 0.5 1" />
+    </material>
+    <material name="red">
+        <color rgba="1 0 0 1" />
+    </material>
+    <material name="green">
+        <color rgba="0 1 0 1"/>
     </material>
     <!--start link llllllllllllllllllllllllllllllllllllllllllllllllllll -->
@@ -36,26 +42,6 @@
         <material>Gazebo/White</material>
     </gazebo>
-    <link name="lidar">
-        <visual>
-            <geometry>
-                <cylinder radius="0.1" length="0.05"/>
-            </geometry>
-            <origin xyz="0 0 0" rpy="0 0 0"/>
-            <material name="black"/>
-        </visual>
-        <collision>
-            <geometry>
-                <cylinder radius="0.1" length="0.05"/>
-            </geometry>
-            <origin xyz="0 0 0" rpy="0 0 0"/>
-        </collision>
-        <xacro:inertial_cylinder mass="0.2" radius="0.1" length="0.05">
-              <origin xyz="0 0 0" rpy="0 0 0"/>
-        </xacro:inertial_cylinder>
-    </link>
-    <gazebo reference="lidar">
-        <material>Gazebo/Black</material>
-    </gazebo>
-    <link name="whil_wright">
+ <!-- right wheeel -->
+    <link name="right_wheel">
       <visual>
           <geometry>
@@ -75,8 +61,9 @@
       </xacro:inertial_cylinder>
     </link>
-    <gazebo reference="whil_wright">
+    <gazebo reference="right_wheel">
         <material>Gazebo/Blue</material>
     </gazebo>
-    <link name="whil_left">
+<!-- left wheeeel -->
+    <link name="left_wheel">
         <visual>
             <geometry>
@@ -96,5 +83,5 @@
         </xacro:inertial_cylinder>
     </link>
-    <gazebo reference="whil_left">
+    <gazebo reference="left_wheel">
         <material>Gazebo/Blue</material>
     </gazebo>
@@ -122,18 +109,13 @@
     </gazebo>
 <!--lllllllllllllllllllllllllllllllllllllllllllllllllllllllllllllllllllllllink eded lllllllllllllllllllllllllllllllllll-->
-    <joint name="base_lidar_joint" type="fixed">
+    <joint name="base_right_wheel_joint" type="continuous">
         <parent link="base_link"/>
-        <child link="lidar"/>
-        <origin xyz="0 0 0.225" rpy="0 0 0"/>
-    </joint>
-    <joint name="base_whil_wright_joint" type="continuous">
-        <parent link="base_link"/>
-        <child link="whil_wright"/>
+        <child link="right_wheel"/>
         <origin xyz="-0.15 -0.225 0" rpy="0 0 0"/>
         <axis xyz="0 1 0"/>
     </joint>
-    <joint name="base_whil_left_joint" type="continuous">
+    <joint name="base_left_wheel_joint" type="continuous">
         <parent link="base_link"/>
-        <child link="whil_left"/>
+        <child link="left_wheel"/>
         <origin xyz="-0.15 0.225 0" rpy="0 0 0"/>
         <axis xyz="0 1 0"/>

File: description/gazebo_control.xacro (robot description, xacro)
@@ -4,6 +4,6 @@
         <plugin name="diff_drive" filename="libgazebo_ros_diff_drive.so">
             <!-- wheel information-->
-            <left_joint>base_whil_left_joint</left_joint>
-            <right_joint>base_whil_wright_joint</right_joint>
+            <left_joint>base_left_wheel_joint</left_joint>
+            <right_joint>base_right_wheel_joint</right_joint>
             <wheel_separation>0.51</wheel_separation>
             <wheel_diameter>0.1</wheel_diameter>

File: description/robot.urdf.xacro (robot description, xacro)
@@ -1,5 +1,14 @@
 <?xml version="1.0"?>
 <robot xmlns:xacro="http://www.ros.org/wiki/xacro" name="robot">
+  <xacro:arg name="use_ros2_control" default="true"/>
   <xacro:include filename="base_robot.xacro" />
-  <xacro:include filename="gazebo_control.xacro" />
+  <xacro:if value="$(arg use_ros2_control)">
+      <xacro:include filename="ros2_control.xacro" />
+  </xacro:if>
+  <xacro:unless value="$(arg use_ros2_control)">
+      <xacro:include filename="gazebo_control.xacro" />
+  </xacro:unless>
+  <xacro:include filename="lidar.xacro"/>
+  <xacro:include filename="camera.xacro"/>
+  <!-- <xacro:include filename="depth_camera.xacro"/> -->
 </robot>
